File: Y11025HL-FLOW_GROVE.kicad_pcb (KiCad board)
At the start: 2 copper layers, 25 x 25.7 mm, 25 parts, among them J1 Grove UART, P2 JTAG, U1 dspic33ep256gp502-QFN, U2 MIC5219-2.6

Commit message: cleaned
Parts:
- added G5: LOGO, xetalsymbols:Xetal-Logo_6.7mm_SilkScreen, B.Cu at (100.1, 91.3)
